File: hardware/board/board.sch (KiCad schematic (older format))
At the start: 38 parts, among them J1 Power, J10 OUT B3, J11 OUT B4, J2 IN A, J3 OUT A1, J4 OUT A2, J5 OUT A3, J6 OUT A4, J7 IN B, J8 OUT B1, J9 OUT B2, U1 OPA4991, U2 OPA4991, U3 LM358

Commit message: Update resistor values; create PDF
Parts:
- R1, R2, R3, R4, R5, R6, R7, R8: value 100R -> 50R; Notes thin film -> thin film, highest possible wattage for size; mpn R0816P-101-D -> (none)
Changed lines of the file:
@@
 P 2975 1500
 F 0 "R1" V 2770 1500 50  0000 C CNN
-F 1 "100R" V 2861 1500 50  0000 C CNN
+F 1 "50R" V 2861 1500 50  0000 C CNN
 F 2 "Resistor_SMD:R_0603_1608Metric_Pad0.98x0.95mm_HandSolder" V 3015 1490 50  0001 C CNN
 F 3 "~" H 2975 1500 50  0001 C CNN
-F 4 "R0816P-101-D" H 2975 1500 50  0001 C CNN "mpn"
-F 5 "thin film" H 2975 1500 50  0001 C CNN "Notes"
+F 4 "" H 2975 1500 50  0001 C CNN "mpn"
+F 5 "thin film, highest possible wattage for size" H 2975 1500 50  0001 C CNN "Notes"
 	1    2975 1500
 	0    1    1    0
@@
 P 2975 2375
 F 0 "R2" V 2770 2375 50  0000 C CNN
-F 1 "100R" V 2861 2375 50  0000 C CNN
+F 1 "50R" V 2861 2375 50  0000 C CNN
 F 2 "Resistor_SMD:R_0603_1608Metric_Pad0.98x0.95mm_HandSolder" V 3015 2365 50  0001 C CNN
 F 3 "~" H 2975 2375 50  0001 C CNN
-F 4 "R0816P-101-D" H 2975 2375 50  0001 C CNN "mpn"
-F 5 "thin film" H 2975 2375 50  0001 C CNN "Notes"
+F 4 "" H 2975 2375 50  0001 C CNN "mpn"
+F 5 "thin film, highest possible wattage for size" H 2975 2375 50  0001 C CNN "Notes"
 	1    2975 2375
 	0    1    1    0
@@
 P 2975 3225
 F 0 "R3" V 2770 3225 50  0000 C CNN
-F 1 "100R" V 2861 3225 50  0000 C CNN
+F 1 "50R" V 2861 3225 50  0000 C CNN
 F 2 "Resistor_SMD:R_0603_1608Metric_Pad0.98x0.95mm_HandSolder" V 3015 3215 50  0001 C CNN
 F 3 "~" H 2975 3225 50  0001 C CNN
-F 4 "R0816P-101-D" H 2975 3225 50  0001 C CNN "mpn"
-F 5 "thin film" H 2975 3225 50  0001 C CNN "Notes"
+F 4 "" H 2975 3225 50  0001 C CNN "mpn"
+F 5 "thin film, highest possible wattage for size" H 2975 3225 50  0001 C CNN "Notes"
 	1    2975 3225
 	0    1    1    0
@@
 P 2975 4125
 F 0 "R4" V 2770 4125 50  0000 C CNN
-F 1 "100R" V 2861 4125 50  0000 C CNN
+F 1 "50R" V 2861 4125 50  0000 C CNN
 F 2 "Resistor_SMD:R_0603_1608Metric_Pad0.98x0.95mm_HandSolder" V 3015 4115 50  0001 C CNN
 F 3 "~" H 2975 4125 50  0001 C CNN
-F 4 "R0816P-101-D" H 2975 4125 50  0001 C CNN "mpn"
-F 5 "thin film" H 2975 4125 50  0001 C CNN "Notes"
+F 4 "" H 2975 4125 50  0001 C CNN "mpn"
+F 5 "thin film, highest possible wattage for size" H 2975 4125 50  0001 C CNN "Notes"
 	1    2975 4125
 	0    1    1    0
@@
 P 7225 1500
 F 0 "R5" V 7020 1500 50  0000 C CNN
-F 1 "100R" V 7111 1500 50  0000 C CNN
+F 1 "50R" V 7111 1500 50  0000 C CNN
 F 2 "Resistor_SMD:R_0603_1608Metric_Pad0.98x0.95mm_HandSolder" V 7265 1490 50  0001 C CNN
 F 3 "~" H 7225 1500 50  0001 C CNN
-F 4 "R0816P-101-D" H 7225 1500 50  0001 C CNN "mpn"
-F 5 "thin film" H 7225 1500 50  0001 C CNN "Notes"
+F 4 "" H 7225 1500 50  0001 C CNN "mpn"
+F 5 "thin film, highest possible wattage for size" H 7225 1500 50  0001 C CNN "Notes"
 	1    7225 1500
 	0    1    1    0
@@
 P 7225 2375
 F 0 "R6" V 7020 2375 50  0000 C CNN
-F 1 "100R" V 7111 2375 50  0000 C CNN
+F 1 "50R" V 7111 2375 50  0000 C CNN
 F 2 "Resistor_SMD:R_0603_1608Metric_Pad0.98x0.95mm_HandSolder" V 7265 2365 50  0001 C CNN
 F 3 "~" H 7225 2375 50  0001 C CNN
-F 4 "R0816P-101-D" H 7225 2375 50  0001 C CNN "mpn"
-F 5 "thin film" H 7225 2375 50  0001 C CNN "Notes"
+F 4 "" H 7225 2375 50  0001 C CNN "mpn"
+F 5 "thin film, highest possible wattage for size" H 7225 2375 50  0001 C CNN "Notes"
 	1    7225 2375
 	0    1    1    0
@@
 P 7225 3225
 F 0 "R7" V 7020 3225 50  0000 C CNN
-F 1 "100R" V 7111 3225 50  0000 C CNN
+F 1 "50R" V 7111 3225 50  0000 C CNN
 F 2 "Resistor_SMD:R_0603_1608Metric_Pad0.98x0.95mm_HandSolder" V 7265 3215 50  0001 C CNN
 F 3 "~" H 7225 3225 50  0001 C CNN
-F 4 "R0816P-101-D" H 7225 3225 50  0001 C CNN "mpn"
-F 5 "thin film" H 7225 3225 50  0001 C CNN "Notes"
+F 4 "" H 7225 3225 50  0001 C CNN "mpn"
+F 5 "thin film, highest possible wattage for size" H 7225 3225 50  0001 C CNN "Notes"
 	1    7225 3225
 	0    1    1    0
@@
 P 7225 4125
 F 0 "R8" V 7020 4125 50  0000 C CNN
-F 1 "100R" V 7111 4125 50  0000 C CNN
+F 1 "50R" V 7111 4125 50  0000 C CNN
 F 2 "Resistor_SMD:R_0603_1608Metric_Pad0.98x0.95mm_HandSolder" V 7265 4115 50  0001 C CNN
 F 3 "~" H 7225 4125 50  0001 C CNN
-F 4 "R0816P-101-D" H 7225 4125 50  0001 C CNN "mpn"
-F 5 "thin film" H 7225 4125 50  0001 C CNN "Notes"
+F 4 "" H 7225 4125 50  0001 C CNN "mpn"
+F 5 "thin film, highest possible wattage for size" H 7225 4125 50  0001 C CNN "Notes"
 	1    7225 4125
 	0    1    1    0

Commit message: Update resistor values
Parts:
- R10, R9: value 270R -> 1.5k; mpn ERJ-3GEYJ271V -> ERJ-3GEYJ1R5V
Changed lines of the file:
@@
 P 2250 5375
 F 0 "R9" H 2182 5329 50  0000 R CNN
-F 1 "270R" H 2182 5420 50  0000 R CNN
+F 1 "1.5k" H 2182 5420 50  0000 R CNN
 F 2 "Resistor_SMD:R_0603_1608Metric_Pad0.98x0.95mm_HandSolder" V 2290 5365 50  0001 C CNN
 F 3 "~" H 2250 5375 50  0001 C CNN
-F 4 "ERJ-3GEYJ271V" H 2250 5375 50  0001 C CNN "mpn"
+F 4 "ERJ-3GEYJ1R5V" H 2250 5375 50  0001 C CNN "mpn"
 F 5 "" H 2250 5375 50  0001 C CNN "unit cost"
 F 6 "5%, thick film" H 2250 5375 50  0001 C CNN "Notes"
@@
 P 6500 5375
 F 0 "R10" H 6432 5329 50  0000 R CNN
-F 1 "270R" H 6432 5420 50  0000 R CNN
+F 1 "1.5k" H 6432 5420 50  0000 R CNN
 F 2 "Resistor_SMD:R_0603_1608Metric_Pad0.98x0.95mm_HandSolder" V 6540 5365 50  0001 C CNN
 F 3 "~" H 6500 5375 50  0001 C CNN
-F 4 "ERJ-3GEYJ271V" H 6500 5375 50  0001 C CNN "mpn"
+F 4 "ERJ-3GEYJ1R5V" H 6500 5375 50  0001 C CNN "mpn"
 F 5 "" H 6500 5375 50  0001 C CNN "unit cost"
 F 6 "5%, thick film" H 6500 5375 50  0001 C CNN "Notes"

Commit message: hardware: add data to schematic for showing parts in the surface mount assembly guide
Parts:
- C1, C2, C3, C4, C5, C6, D1, D2, D3, D4, D5, D6, FB1, FB2, R1, R10, R2, R3, R4, R5, R6, R7, R8, R9, U1, U2, U3: smd kit (none) -> yes
Changed lines of the file:
@@
 F 4 "" H 2975 1500 50  0001 C CNN "mpn"
 F 5 "thin film, highest possible wattage for size" H 2975 1500 50  0001 C CNN "Notes"
+F 6 "yes" H 2975 1500 50  0001 C CNN "smd kit"
 	1    2975 1500
 	0    1    1    0
@@
 F 4 "OPA4991IPWR " H 2525 2375 50  0001 C CNN "mpn"
 F 5 "" H 2525 2375 50  0001 C CNN "unit cost"
+F 6 "yes" H 2525 2375 50  0001 C CNN "smd kit"
 	2    2525 2375
 	1    0    0    -1
@@
 F 4 "" H 2975 2375 50  0001 C CNN "mpn"
 F 5 "thin film, highest possible wattage for size" H 2975 2375 50  0001 C CNN "Notes"
+F 6 "yes" H 2975 2375 50  0001 C CNN "smd kit"
 	1    2975 2375
 	0    1    1    0
@@
 F 4 "OPA4991IPWR " H 2525 3225 50  0001 C CNN "mpn"
 F 5 "" H 2525 3225 50  0001 C CNN "unit cost"
+F 6 "yes" H 2525 3225 50  0001 C CNN "smd kit"
 	1    2525 3225
 	1    0    0    -1
@@
 F 4 "" H 2975 3225 50  0001 C CNN "mpn"
 F 5 "thin film, highest possible wattage for size" H 2975 3225 50  0001 C CNN "Notes"
+F 6 "yes" H 2975 3225 50  0001 C CNN "smd kit"
 	1    2975 3225
 	0    1    1    0
@@
 F 4 "" H 2975 4125 50  0001 C CNN "mpn"
 F 5 "thin film, highest possible wattage for size" H 2975 4125 50  0001 C CNN "Notes"
+F 6 "yes" H 2975 4125 50  0001 C CNN "smd kit"
 	1    2975 4125
 	0    1    1    0
@@
 F 4 "OPA4991IPWR " H 6775 1500 50  0001 C CNN "mpn"
 F 5 "" H 6775 1500 50  0001 C CNN "unit cost"
+F 6 "yes" H 6775 1500 50  0001 C CNN "smd kit"
 	4    6775 1500
 	1    0    0    -1
@@
 F 4 "" H 7225 1500 50  0001 C CNN "mpn"
 F 5 "thin film, highest possible wattage for size" H 7225 1500 50  0001 C CNN "Notes"
+F 6 "yes" H 7225 1500 50  0001 C CNN "smd kit"
 	1    7225 1500
 	0    1    1    0
@@
 F 4 "OPA4991IPWR " H 6775 2375 50  0001 C CNN "mpn"
 F 5 "" H 6775 2375 50  0001 C CNN "unit cost"
+F 6 "yes" H 6775 2375 50  0001 C CNN "smd kit"
 	3    6775 2375
 	1    0    0    -1
@@
 F 4 "" H 7225 2375 50  0001 C CNN "mpn"
 F 5 "thin film, highest possible wattage for size" H 7225 2375 50  0001 C CNN "Notes"
+F 6 "yes" H 7225 2375 50  0001 C CNN "smd kit"
 	1    7225 2375
 	0    1    1    0
@@
 F 4 "OPA4991IPWR " H 6775 3225 50  0001 C CNN "mpn"
 F 5 "" H 6775 3225 50  0001 C CNN "unit cost"
+F 6 "yes" H 6775 3225 50  0001 C CNN "smd kit"
 	4    6775 3225
 	1    0    0    -1
@@
 F 4 "" H 7225 3225 50  0001 C CNN "mpn"
 F 5 "thin film, highest possible wattage for size" H 7225 3225 50  0001 C CNN "Notes"
+F 6 "yes" H 7225 3225 50  0001 C CNN "smd kit"
 	1    7225 3225
 	0    1    1    0
@@
 F 4 "OPA4991IPWR " H 6775 4125 50  0001 C CNN "mpn"
 F 5 "" H 6775 4125 50  0001 C CNN "unit cost"
+F 6 "yes" H 6775 4125 50  0001 C CNN "smd kit"
 	3    6775 4125
 	1    0    0    -1
@@
 F 4 "" H 7225 4125 50  0001 C CNN "mpn"
 F 5 "thin film, highest possible wattage for size" H 7225 4125 50  0001 C CNN "Notes"
+F 6 "yes" H 7225 4125 50  0001 C CNN "smd kit"
 	1    7225 4125
 	0    1    1    0
@@
 F 5 "" H 2450 6800 50  0001 C CNN "unit cost"
 F 6 "300mA" H 2450 6800 50  0001 C CNN "Notes"
+F 7 "yes" H 2450 6800 50  0001 C CNN "smd kit"
 	1    2450 6800
 	0    1    1    0
@@
 F 5 "" H 3025 6800 50  0001 C CNN "unit cost"
 F 6 "Any PMEGxxxxEGW part, 500mA If" H 3025 6800 50  0001 C CNN "Notes"
+F 7 "yes" H 3025 6800 50  0001 C CNN "smd kit"
 	1    3025 6800
 	1    0    0    -1
@@
 F 4 "OPA4991IPWR " H 8475 5575 50  0001 C CNN "mpn"
 F 5 "" H 8475 6025 50  0001 C CNN "unit cost"
+F 6 "yes" H 8475 6025 50  0001 C CNN "smd kit"
 	5    8475 6025
 	1    0    0    -1
@@
 F 4 "OPA4991IPWR " H 9350 6025 50  0001 C CNN "mpn"
 F 5 "" H 9350 6025 50  0001 C CNN "unit cost"
+F 6 "yes" H 9350 6025 50  0001 C CNN "smd kit"
 	5    9350 6025
 	1    0    0    -1
@@
 F 5 "" H 2450 7300 50  0001 C CNN "unit cost"
 F 6 "300mA" H 2450 7300 50  0001 C CNN "Notes"
+F 7 "yes" H 2450 7300 50  0001 C CNN "smd kit"
 	1    2450 7300
 	0    1    1    0
@@
 F 5 "" H 3025 7300 50  0001 C CNN "unit cost"
 F 6 "Any PMEGxxxxEGW part, 500mA If" H 3025 7300 50  0001 C CNN "Notes"
+F 7 "yes" H 3025 7300 50  0001 C CNN "smd kit"
 	1    3025 7300
 	-1   0    0    1
@@
 F 5 "" H 9800 5750 50  0001 C CNN "unit cost"
 F 6 "0603, 25V+, 10%, Bypass cap" H 9800 5750 50  0001 C CNN "Notes"
+F 7 "yes" H 9800 5750 50  0001 C CNN "smd kit"
 	1    9800 5750
 	1    0    0    -1
@@
 F 5 "" H 10150 5750 50  0001 C CNN "unit cost"
 F 6 "0603, 25V+, 10%, Bypass cap" H 10150 5750 50  0001 C CNN "Notes"
+F 7 "yes" H 10150 5750 50  0001 C CNN "smd kit"
 	1    10150 5750
 	1    0    0    -1
@@
 F 5 "" H 9800 6375 50  0001 C CNN "unit cost"
 F 6 "0603, 25V+, 10%, Bypass cap" H 9800 6375 50  0001 C CNN "Notes"
+F 7 "yes" H 9800 6375 50  0001 C CNN "smd kit"
 	1    9800 6375
 	1    0    0    -1
@@
 F 5 "" H 10150 6375 50  0001 C CNN "unit cost"
 F 6 "0603, 25V+, 10%, Bypass cap" H 10150 6375 50  0001 C CNN "Notes"
+F 7 "yes" H 10150 6375 50  0001 C CNN "smd kit"
 	1    10150 6375
 	1    0    0    -1
@@
 F 5 "" H 3900 7075 50  0001 C CNN "unit cost"
 F 6 "0805, 25V+, 10%, Bulk cap" H 3900 7075 50  0001 C CNN "Notes"
+F 7 "yes" H 3900 7075 50  0001 C CNN "smd kit"
 	1    3900 7075
 	1    0    0    -1
@@
 F 5 "" H 4300 7050 50  0001 C CNN "unit cost"
 F 6 "0805, 25V+, 10%, Bulk cap" H 4300 7050 50  0001 C CNN "Notes"
+F 7 "yes" H 4300 7050 50  0001 C CNN "smd kit"
 	1    4300 7050
 	-1   0    0    1
@@
 F 4 "OPA4991IPWR " H 2525 4125 50  0001 C CNN "mpn"
 F 5 "" H 2525 4125 50  0001 C CNN "unit cost"
+F 6 "yes" H 2525 4125 50  0001 C CNN "smd kit"
 	2    2525 4125
 	1    0    0    -1
@@
 F 4 "LM358PWR" H 2550 4900 50  0001 C CNN "mpn"
 F 5 "" H 2550 4900 50  0001 C CNN "unit cost"
+F 6 "yes" H 2550 4900 50  0001 C CNN "smd kit"
 	2    2550 4900
 	1    0    0    -1
@@
 F 5 "" H 2975 5075 50  0001 C CNN "unit cost"
 F 6 "Red" H 2975 5075 50  0001 C CNN "Notes"
+F 7 "yes" H 2975 5075 50  0001 C CNN "smd kit"
 	1    2975 5075
 	0    1    1    0
@@
 F 5 "" H 2850 5075 50  0001 C CNN "unit cost"
 F 6 "Blue" H 2850 5075 50  0001 C CNN "Notes"
+F 7 "yes" H 2850 5075 50  0001 C CNN "smd kit"
 	1    2850 5075
 	0    -1   -1   0
@@
 F 5 "" H 2250 5375 50  0001 C CNN "unit cost"
 F 6 "5%, thick film" H 2250 5375 50  0001 C CNN "Notes"
+F 7 "yes" H 2250 5375 50  0001 C CNN "smd kit"
 	1    2250 5375
 	-1   0    0    1
@@
 F 4 "LM358PWR" H 6800 4900 50  0001 C CNN "mpn"
 F 5 "" H 6800 4900 50  0001 C CNN "unit cost"
+F 6 "yes" H 6800 4900 50  0001 C CNN "smd kit"
 	1    6800 4900
 	1    0    0    -1
@@
 F 5 "" H 7225 5075 50  0001 C CNN "unit cost"
 F 6 "Red" H 7225 5075 50  0001 C CNN "Notes"
+F 7 "yes" H 7225 5075 50  0001 C CNN "smd kit"
 	1    7225 5075
 	0    1    1    0
@@
 F 5 "" H 7100 5075 50  0001 C CNN "unit cost"
 F 6 "Blue" H 7100 5075 50  0001 C CNN "Notes"
+F 7 "yes" H 7100 5075 50  0001 C CNN "smd kit"
 	1    7100 5075
 	0    -1   -1   0
@@
 F 5 "" H 6500 5375 50  0001 C CNN "unit cost"
 F 6 "5%, thick film" H 6500 5375 50  0001 C CNN "Notes"
+F 7 "yes" H 6500 5375 50  0001 C CNN "smd kit"
 	1    6500 5375
 	-1   0    0    1
@@
 F 4 "LM358PWR" H 7825 6025 50  0001 C CNN "mpn"
 F 5 "" H 7825 6025 50  0001 C CNN "unit cost"
+F 6 "yes" H 7825 6025 50  0001 C CNN "smd kit"
 	3    7825 6025
 	1    0    0    -1
@@
 F 4 "OPA4991IPWR " H 2525 1500 50  0001 C CNN "mpn"
 F 5 "" H 2525 1500 50  0001 C CNN "unit cost"
+F 6 "yes" H 2525 1500 50  0001 C CNN "smd kit"
 	1    2525 1500
 	1    0    0    -1
